Commit message: edits to folder name

File: robot_description_mai_mohsen/urdf/robot_description.urdf.xacro (robot description, xacro)
@@ -1,4 +1,5 @@
 <?xml version="1.0"?>
 <robot name="two_wheeled_robot" xmlns:xacro="http://www.ros.org/wiki/xacro">
+<xacro:arg name="mesh_path" default="package://my_robot_description/meshes/"/>
   <xacro:property name="base_length" value="0.6"/>
   <xacro:property name="base_width" value="0.4"/>
@@ -111,5 +112,5 @@
       <origin xyz="0 0 0" rpy="0 0 0"/>
       <geometry>
-        <mesh filename="../meshes/lidar.STL"/>
+        <mesh filename="$(arg mesh_path)lidar.STL"/>
       </geometry>
       <material name="lidar_gray">
@@ -136,5 +137,5 @@
     <visual>
       <geometry>
-        <mesh filename="../meshes/zed.stl"/>
+        <mesh filename="$(arg mesh_path)zed.stl"/>
       </geometry>
       <material name="camera_color">
